Commit message: final

File: src/rover_description/robots/rover.urdf.xacro (robot description, xacro)
@@ -1,182 +1,168 @@
-<?xml version="1.0" ?>
-<robot name="rover"
-    xmlns:xacro="http://www.ros.org/wiki/xacro">
-    <!-- Include macros -->
-    <xacro:include filename="$(find rover_description)/urdf/materials.xacro"/>
-    <xacro:include filename="$(find rover_description)/urdf/inertials.xacro"/>
-    <xacro:include filename="$(find rover_description)/urdf/bases/body.urdf.xacro" />
-    <xacro:include filename="$(find rover_description)/urdf/bases/differential.urdf.xacro" />
-    <xacro:include filename="$(find rover_description)/urdf/bases/turnbuckle.urdf.xacro" />
-    <xacro:include filename="$(find rover_description)/urdf/bases/rocker.urdf.xacro" />
-    <xacro:include filename="$(find rover_description)/urdf/bases/bogie.urdf.xacro" />
-    <xacro:include filename="$(find rover_description)/urdf/wheels/wheel.urdf.xacro" />
-    <xacro:include filename="$(find rover_description)/urdf/wheels/corner.urdf.xacro" />
-    <xacro:include filename="$(find rover_description)/urdf/sensors/all_sensors.urdf.xacro" />
-        <gazebo>
-        <plugin filename="gz_ros2_control-system" name="gz_ros2_control::GazeboSimROS2ControlPlugin">
-            <parameters>$(find rover_description)/config/control.yaml</parameters>
-            <ros>
-                <namespace>/</namespace>
-            </ros>
-        </plugin>
-        <plugin filename="libignition-gazebo-sensors-system.so" name="ignition::gazebo::systems::Sensors">
-            <render_engine>ogre2</render_engine>
-        </plugin>
-        <plugin filename="libignition-gazebo-imu-system.so" name="ignition::gazebo::systems::Imu">
-        </plugin>
-    </gazebo>
-    <ros2_control name="IgnitionSystem" type="system">
-        <hardware>
-            <plugin>gz_ros2_control/GazeboSimSystem</plugin>
-        </hardware>
-        <joint name="front_right_corner_joint">
-            <command_interface name="position">
-                <param name="min">-3.14159</param>
-                <param name="max">3.14159</param>
-            </command_interface>
-            <state_interface name="position">
-                <param name="initial_value">0.0</param>
-            </state_interface>
-            <state_interface name="velocity"/>
-            <state_interface name="effort"/>
-        </joint>
-        <joint name="front_left_corner_joint">
-            <command_interface name="position">
-                <param name="min">-3.14159</param>
-                <param name="max">3.14159</param>
-            </command_interface>
-            <state_interface name="position">
-                <param name="initial_value">0.0</param>
-            </state_interface>
-            <state_interface name="velocity"/>
-            <state_interface name="effort"/>
-        </joint>
-        <joint name="back_right_corner_joint">
-            <command_interface name="position">
-                <param name="min">-3.14159</param>
-                <param name="max">3.14159</param>
-            </command_interface>
-            <state_interface name="position">
-                <param name="initial_value">0.0</param>
-            </state_interface>
-            <state_interface name="velocity"/>
-            <state_interface name="effort"/>
-        </joint>
-        <joint name="back_left_corner_joint">
-            <command_interface name="position">
-                <param name="min">-3.14159</param>
-                <param name="max">3.14159</param>
-            </command_interface>
-            <state_interface name="position">
-                <param name="initial_value">0.0</param>
-            </state_interface>
-            <state_interface name="velocity"/>
-            <state_interface name="effort"/>
-        </joint>
-        <joint name="front_right_wheel_joint">
-            <command_interface name="velocity">
-                <param name="min">-10</param>
-                <param name="max">10</param>
-            </command_interface>
-            <state_interface name="position"/>
-            <state_interface name="velocity"/>
-            <state_interface name="effort"/>
-        </joint>
-        <joint name="front_left_wheel_joint">
-            <command_interface name="velocity">
-                <param name="min">-10</param>
-                <param name="max">10</param>
-            </command_interface>
-            <state_interface name="position"/>
-            <state_interface name="velocity"/>
-            <state_interface name="effort"/>
-        </joint>
-        <joint name="mid_right_wheel_joint">
-            <command_interface name="velocity">
-                <param name="min">-10</param>
-                <param name="max">10</param>
-            </command_interface>
-            <state_interface name="position"/>
-            <state_interface name="velocity"/>
-            <state_interface name="effort"/>
-        </joint>
-        <joint name="mid_left_wheel_joint">
-            <command_interface name="velocity">
-                <param name="min">-10</param>
-                <param name="max">10</param>
-            </command_interface>
-            <state_interface name="position"/>
-            <state_interface name="velocity"/>
-            <state_interface name="effort"/>
-        </joint>
-        <joint name="back_right_wheel_joint">
-            <command_interface name="velocity">
-                <param name="min">-10</param>
-                <param name="max">10</param>
-            </command_interface>
-            <state_interface name="position"/>
-            <state_interface name="velocity"/>
-            <state_interface name="effort"/>
-        </joint>
-        <joint name="back_left_wheel_joint">
-            <command_interface name="velocity">
-                <param name="min">-10</param>
-                <param name="max">10</param>
-            </command_interface>
-            <state_interface name="position"/>
-            <state_interface name="velocity"/>
-            <state_interface name="effort"/>
-        </joint>
-    </ros2_control>
-    <!-- The base link -->
-    <link name="base_link">
-        <visual>
-            <origin rpy="0 0 0" xyz="0 0 0" />
-            <geometry>
-                <box size="0.01 0.01 0.01"/>
-            </geometry>
-            <material name="orange" />
-        </visual>
-    </link>
-    <gazebo reference="base_link">
-        <material>Gazebo/Orange</material>
-    </gazebo>
-    <!-- body -->
-    <xacro:body parent="base_link" />
-    <xacro:differential parent="base_link" />
-    <xacro:rocker parent="base_link" lat_label="left" reflect="1"/>
-    <xacro:rocker parent="base_link" lat_label="right" reflect="-1"/>
-    <xacro:bogie lat_label="left" reflect="1"/>
-    <xacro:bogie lat_label="right" reflect="-1"/>
-    <!-- sensors -->
-    <xacro:sensor_hokuyo prefix="laser" parent="base_link" min_angle="-1.0" max_angle="1.0">
-        <origin xyz="0.17 0 0.005" rpy="0 0 0"/>
-    </xacro:sensor_hokuyo>
-    <xacro:sensor_imu prefix="imu" parent="base_link">
-        <origin xyz="0 0 -0.04" rpy="0 0 0"/>
-    </xacro:sensor_imu>
-    <xacro:sensor_asus_xtion prefix="camera" parent="base_link">
-        <origin xyz="0.215 0 0.065" rpy="0 0.15 0"/>
-    </xacro:sensor_asus_xtion>
-    <!-- wheels -->
-    <xacro:corner_link lon_label="front" lat_label="left" reflect="1"/>
-    <xacro:corner_link lon_label="front" lat_label="right" reflect="-1"/>
-    <xacro:front_corner_joint lat_label="left" reflect="1"/>
-    <xacro:front_corner_joint lat_label="right" reflect="-1"/>
-    <xacro:corner_link lon_label="back" lat_label="left" reflect="1"/>
-    <xacro:corner_link lon_label="back" lat_label="right" reflect="-1"/>
-    <xacro:back_corner_joint lat_label="left" reflect="1"/>
-    <xacro:back_corner_joint lat_label="right" reflect="-1"/>
-    <xacro:wheel_link lon_label="front" lat_label="left" reflect="1"/>
-    <xacro:wheel_link lon_label="front" lat_label="right" reflect="-1"/>
-    <xacro:corner_wheel_joint lon_label="front" lat_label="left" reflect="1"/>
-    <xacro:corner_wheel_joint lon_label="front" lat_label="right" reflect="-1"/>
-    <xacro:wheel_link lon_label="mid" lat_label="left" reflect="1"/>
-    <xacro:wheel_link lon_label="mid" lat_label="right" reflect="-1"/>
-    <xacro:mid_wheel_joint lat_label="left" reflect="1"/>
-    <xacro:mid_wheel_joint lat_label="right" reflect="-1"/>
-    <xacro:wheel_link lon_label="back" lat_label="left" reflect="1"/>
-    <xacro:wheel_link lon_label="back" lat_label="right" reflect="-1"/>
-    <xacro:corner_wheel_joint lon_label="back" lat_label="left" reflect="1"/>
-    <xacro:corner_wheel_joint lon_label="back" lat_label="right" reflect="-1"/>
-</robot>
+<ros2_control name="IgnitionSystem" type="system">
+    <hardware>
+        <plugin>gz_ros2_control/GazeboSimSystem</plugin>
+    </hardware>
+    <!-- ================= Steering Joints ================= -->
+    <joint name="front_right_corner_joint">
+        <command_interface name="position">
+            <!-- ==========================================================
+                TODO 1 — Configure Steering Angle Limits
+                Parameters:
+                  min
+                  max
+                Controls:
+                  Defines the minimum and maximum steering angle that
+                  can be commanded to each steering joint.
+                Why is this important?
+                  These limits determine how far the front and rear
+                  steering wheels are allowed to rotate. Any steering
+                  command outside this range will be clipped by the
+                  controller.
+                Effects:
+                • Larger limits:
+                    - Enables tighter turns.
+                    - May produce unrealistic steering if set too high.
+                • Smaller limits:
+                    - Produces smoother steering.
+                    - Increases the rover's turning radius.
+                Hint:
+                - Use values in radians.
+                - The limits should be symmetric (±θ).
+                - Most mobile robots use steering limits between
+                  ±0.5 and ±1.2 radians.
+            ========================================================== -->
+            <param name="min"># TODO</param>
+            <param name="max"># TODO</param>
+        </command_interface>
+        <state_interface name="position">
+            <param name="initial_value">0.0</param>
+        </state_interface>
+        <state_interface name="velocity"/>
+        <state_interface name="effort"/>
+    </joint>
+    <!--
+      NOTE:
+      Apply the same steering limits to the remaining steering joints
+      to maintain symmetric steering behaviour.
+    -->
+    <joint name="front_left_corner_joint">
+        <command_interface name="position">
+            <param name="min"># TODO</param>
+            <param name="max"># TODO</param>
+        </command_interface>
+        <state_interface name="position">
+            <param name="initial_value">0.0</param>
+        </state_interface>
+        <state_interface name="velocity"/>
+        <state_interface name="effort"/>
+    </joint>
+    <joint name="back_right_corner_joint">
+        <command_interface name="position">
+            <param name="min"># TODO</param>
+            <param name="max"># TODO</param>
+        </command_interface>
+        <state_interface name="position">
+            <param name="initial_value">0.0</param>
+        </state_interface>
+        <state_interface name="velocity"/>
+        <state_interface name="effort"/>
+    </joint>
+    <joint name="back_left_corner_joint">
+        <command_interface name="position">
+            <param name="min"># TODO</param>
+            <param name="max"># TODO</param>
+        </command_interface>
+        <state_interface name="position">
+            <param name="initial_value">0.0</param>
+        </state_interface>
+        <state_interface name="velocity"/>
+        <state_interface name="effort"/>
+    </joint>
+    <!-- ================= Drive Wheels ================= -->
+    <joint name="front_right_wheel_joint">
+        <command_interface name="velocity">
+            <!-- ==========================================================
+                TODO 2 — Configure Maximum Wheel Speed
+                Parameters:
+                  min
+                  max
+                Controls:
+                  Defines the minimum and maximum rotational velocity
+                  that can be commanded to each drive wheel.
+                Why is this important?
+                  These limits determine the rover's maximum driving
+                  speed. Any velocity command beyond these limits will
+                  automatically be clipped by the controller.
+                Effects:
+                • Larger limits:
+                    - Higher maximum speed.
+                    - Faster mission completion.
+                    - Reduced stability if excessively large.
+                • Smaller limits:
+                    - Slower and smoother motion.
+                    - Easier control.
+                    - Longer travel time.
+                Hint:
+                - Use equal positive and negative limits so the rover
+                  can move both forward and backward.
+                - Units are radians per second (rad/s).
+                - Choose values that balance speed and stability.
+            ========================================================== -->
+            <param name="min"># TODO</param>
+            <param name="max"># TODO</param>
+        </command_interface>
+        <state_interface name="position"/>
+        <state_interface name="velocity"/>
+        <state_interface name="effort"/>
+    </joint>
+    <!--
+      NOTE:
+      Apply the same velocity limits to all remaining drive wheels
+      so every wheel shares the same maximum speed.
+    -->
+    <joint name="front_left_wheel_joint">
+        <command_interface name="velocity">
+            <param name="min"># TODO</param>
+            <param name="max"># TODO</param>
+        </command_interface>
+        <state_interface name="position"/>
+        <state_interface name="velocity"/>
+        <state_interface name="effort"/>
+    </joint>
+    <joint name="mid_right_wheel_joint">
+        <command_interface name="velocity">
+            <param name="min"># TODO</param>
+            <param name="max"># TODO</param>
+        </command_interface>
+        <state_interface name="position"/>
+        <state_interface name="velocity"/>
+        <state_interface name="effort"/>
+    </joint>
+    <joint name="mid_left_wheel_joint">
+        <command_interface name="velocity">
+            <param name="min"># TODO</param>
+            <param name="max"># TODO</param>
+        </command_interface>
+        <state_interface name="position"/>
+        <state_interface name="velocity"/>
+        <state_interface name="effort"/>
+    </joint>
+    <joint name="back_right_wheel_joint">
+        <command_interface name="velocity">
+            <param name="min"># TODO</param>
+            <param name="max"># TODO</param>
+        </command_interface>
+        <state_interface name="position"/>
+        <state_interface name="velocity"/>
+        <state_interface name="effort"/>
+    </joint>
+    <joint name="back_left_wheel_joint">
+        <command_interface name="velocity">
+            <param name="min"># TODO</param>
+            <param name="max"># TODO</param>
+        </command_interface>
+        <state_interface name="position"/>
+        <state_interface name="velocity"/>
+        <state_interface name="effort"/>
+    </joint>
+</ros2_control>
